Commit message: turtlebot3_waffle_pi에 카메라 추가완료

File: src/turtlebot3/turtlebot3_description/urdf/turtlebot3_waffle_pi.gazebo.xacro (robot description, xacro)
@@ -136,5 +136,5 @@
 <!--link : https://www.raspberrypi.org/documentation/hardware/camera/-->
   <gazebo reference="camera_rgb_frame">
-    <sensor type="camera" name="Pi Camera">
+    <sensor type="depth" name="Pi Camera">
       <always_on>true</always_on>
       <visualize>$(arg camera_visual)</visualize>
@@ -146,4 +146,5 @@
               <format>R8G8B8</format>
           </image>
+          <depth_camera></depth_camera>
           <clip>
               <near>0.03</near>
@@ -151,5 +152,6 @@
           </clip>
       </camera>
-      <plugin name="camera_controller" filename="libgazebo_ros_camera.so">
+      <plugin name="camera_controller" filename="libgazebo_ros_openni_kinect.so">
+        <baseline>0.2</baseline>
         <alwaysOn>true</alwaysOn>
         <updateRate>30.0</updateRate>
@@ -157,5 +159,10 @@
         <frameName>camera_rgb_optical_frame</frameName>
         <imageTopicName>rgb/image_raw</imageTopicName>
+        <depthImageTopicName>depth/image_raw</depthImageTopicName>
+        <pointCloudTopicName>depth/points</pointCloudTopicName>
         <cameraInfoTopicName>rgb/camera_info</cameraInfoTopicName>
+        <depthImageCameraInfoTopicName>depth/camera_info</depthImageCameraInfoTopicName>
+        <pointCloudCutoff>0.4</pointCloudCutoff>
+        <pointCloudCutoffMax>8.0</pointCloudCutoffMax>
         <hackBaseline>0.07</hackBaseline>
         <distortionK1>0.0</distortionK1>
@@ -164,4 +171,8 @@
         <distortionT1>0.0</distortionT1>
         <distortionT2>0.0</distortionT2>
+        <CxPrime>0.0</CxPrime>
+        <Cx>0.0</Cx>
+        <Cy>0.0</Cy>
+        <focalLength>0</focalLength>
       </plugin>
     </sensor>

File: src/turtlebot3/turtlebot3_description/urdf/turtlebot3_waffle_pi.urdf.xacro (robot description, xacro)
@@ -166,4 +166,18 @@
   </joint>
   <link name="camera_link">
+    <visual>
+      <origin xyz="0.005 0.011 0.013" rpy="0 0 0"/>
+      <geometry>
+        <box size="0.018 0.034 0.028"/>
+      </geometry>
+      <material name="dark"/>
+    </visual>
+    <visual>
+      <origin xyz="0.016 0.011 0.013" rpy="0 1.5708 0"/>
+      <geometry>
+        <cylinder length="0.006" radius="0.007"/>
+      </geometry>
+      <material name="black"/>
+    </visual>
     <collision>
       <origin xyz="0.005 0.011 0.013" rpy="0 0 0"/>
