Commit message: modified world file, yolo_detection.launch, added yolo_detector.py

File: src/turtlebot3_description/urdf/turtlebot3_burger.urdf.xacro (robot description, xacro)
@@ -149,6 +149,4 @@
         <box size="0.02 0.02 0.02"/>
       </geometry>
-      <!-- 카메라를 검은색으로 표현 -->
-      <material name="black"/>
     </visual>
   </link>
